File: Hardware/PCB/FastConverter/FastConverter.kicad_sch (KiCad schematic)
At the start: 3 parts

Commit message: new: hook up PCB
Parts:
- removed U?: 90DegreePort, port:NEScontrollerport, symbol nescontroller:90DegreePort
- added U2: 90DegreePort, port:NEScontrollerport, symbol nescontroller:90DegreePort
- U3: renamed from U?; footprint (none) -> promicro:ProMicro
- gave numbers to parts that had none: 1
Connections:
- net at U3.10 (E6): now also U2.C (Clock)
- net at U3.21 (VCC): now also U1.5V, U2.5V
- net at U3.3 (GND): now also U1.G (Ground), U2.G (Ground)
- net at U3.5 (SDA): now also U1.D (Data)
- net at U3.6 (SCL): now also U1.L (Latch)
- net at U3.7 (D4): now also U1.C (Clock)
- net at U3.8 (C6): now also U2.D (Data)
- net at U3.9 (D7): now also U2.L (Latch)
Other:
- moved on the sheet: U1, U3
Changed lines of the file:
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@@
 (kicad_sch (version 20211123) (generator eeschema)
   (paper "A4")
-  (symbol (lib_id "promicro:ProMicro") (at 77.47 90.17 0) (unit 1)
+  (junction (at 115.57 78.74) (diameter 0) (color 0 0 0 0)
+  )
+  (junction (at 72.39 76.2) (diameter 0) (color 0 0 0 0)
+  )
+  (wire (pts (xy 48.26 107.95) (xy 74.93 107.95))
+    (stroke (width 0) (type default) (color 0 0 0 0))
+  )
+  (wire (pts (xy 76.2 86.36) (xy 60.96 86.36))
+    (stroke (width 0) (type default) (color 0 0 0 0))
+  )
+  (wire (pts (xy 115.57 62.23) (xy 115.57 78.74))
+    (stroke (width 0) (type default) (color 0 0 0 0))
+  )
+  (wire (pts (xy 71.12 102.87) (xy 71.12 88.9))
+    (stroke (width 0) (type default) (color 0 0 0 0))
+  )
+  (wire (pts (xy 115.57 110.49) (xy 115.57 78.74))
+    (stroke (width 0) (type default) (color 0 0 0 0))
+  )
+  (wire (pts (xy 74.93 93.98) (xy 76.2 93.98))
+    (stroke (width 0) (type default) (color 0 0 0 0))
+  )
+  (wire (pts (xy 66.04 76.2) (xy 72.39 76.2))
+    (stroke (width 0) (type default) (color 0 0 0 0))
+  )
+  (wire (pts (xy 76.2 81.28) (xy 63.5 81.28))
+    (stroke (width 0) (type default) (color 0 0 0 0))
+  )
+  (wire (pts (xy 63.5 81.28) (xy 63.5 67.31))
+    (stroke (width 0) (type default) (color 0 0 0 0))
+  )
+  (wire (pts (xy 69.85 74.93) (xy 69.85 62.23))
+    (stroke (width 0) (type default) (color 0 0 0 0))
+  )
+  (wire (pts (xy 115.57 78.74) (xy 111.76 78.74))
+    (stroke (width 0) (type default) (color 0 0 0 0))
+  )
+  (wire (pts (xy 48.26 64.77) (xy 72.39 64.77))
+    (stroke (width 0) (type default) (color 0 0 0 0))
+  )
+  (wire (pts (xy 48.26 72.39) (xy 60.96 72.39))
+    (stroke (width 0) (type default) (color 0 0 0 0))
+  )
+  (wire (pts (xy 48.26 69.85) (xy 62.23 69.85))
+    (stroke (width 0) (type default) (color 0 0 0 0))
+  )
+  (wire (pts (xy 48.26 105.41) (xy 72.39 105.41))
+    (stroke (width 0) (type default) (color 0 0 0 0))
+  )
+  (wire (pts (xy 48.26 74.93) (xy 69.85 74.93))
+    (stroke (width 0) (type default) (color 0 0 0 0))
+  )
+  (wire (pts (xy 74.93 107.95) (xy 74.93 93.98))
+    (stroke (width 0) (type default) (color 0 0 0 0))
+  )
+  (wire (pts (xy 62.23 83.82) (xy 62.23 69.85))
+    (stroke (width 0) (type default) (color 0 0 0 0))
+  )
+  (wire (pts (xy 63.5 67.31) (xy 48.26 67.31))
+    (stroke (width 0) (type default) (color 0 0 0 0))
+  )
+  (wire (pts (xy 72.39 91.44) (xy 76.2 91.44))
+    (stroke (width 0) (type default) (color 0 0 0 0))
+  )
+  (wire (pts (xy 60.96 86.36) (xy 60.96 72.39))
+    (stroke (width 0) (type default) (color 0 0 0 0))
+  )
+  (wire (pts (xy 48.26 110.49) (xy 115.57 110.49))
+    (stroke (width 0) (type default) (color 0 0 0 0))
+  )
+  (wire (pts (xy 48.26 100.33) (xy 66.04 100.33))
+    (stroke (width 0) (type default) (color 0 0 0 0))
+  )
+  (wire (pts (xy 48.26 102.87) (xy 71.12 102.87))
+    (stroke (width 0) (type default) (color 0 0 0 0))
+  )
+  (wire (pts (xy 66.04 100.33) (xy 66.04 76.2))
+    (stroke (width 0) (type default) (color 0 0 0 0))
+  )
+  (wire (pts (xy 69.85 62.23) (xy 115.57 62.23))
+    (stroke (width 0) (type default) (color 0 0 0 0))
+  )
+  (wire (pts (xy 71.12 88.9) (xy 76.2 88.9))
+    (stroke (width 0) (type default) (color 0 0 0 0))
+  )
+  (wire (pts (xy 72.39 64.77) (xy 72.39 76.2))
+    (stroke (width 0) (type default) (color 0 0 0 0))
+  )
+  (wire (pts (xy 76.2 83.82) (xy 62.23 83.82))
+    (stroke (width 0) (type default) (color 0 0 0 0))
+  )
+  (wire (pts (xy 72.39 105.41) (xy 72.39 91.44))
+    (stroke (width 0) (type default) (color 0 0 0 0))
+  )
+  (wire (pts (xy 72.39 76.2) (xy 76.2 76.2))
+    (stroke (width 0) (type default) (color 0 0 0 0))
+  )
+  (symbol (lib_id "promicro:ProMicro") (at 93.98 90.17 0) (unit 1)
     (in_bom yes) (on_board yes)
-    (property "Reference" "U?" (id 0) (at 77.47 63.8302 0)
+    (property "Reference" "U3" (id 0) (at 93.98 63.8302 0)
       (effects (font (size 1.524 1.524)))
     )
-    (property "Value" "" (id 1) (at 77.47 66.5226 0)
+    (property "Value" "" (id 1) (at 93.98 66.5226 0)
       (effects (font (size 1.524 1.524)))
     )
-    (property "Footprint" "" (id 2) (at 80.01 116.84 0)
+    (property "Footprint" "promicro:ProMicro" (id 2) (at 93.98 102.87 0)
       (effects (font (size 1.524 1.524)))
     )
-    (property "Datasheet" "" (id 3) (at 80.01 116.84 0)
+    (property "Datasheet" "" (id 3) (at 96.52 116.84 0)
       (effects (font (size 1.524 1.524)))
     )
@@
     (pin "9")
   )
-  (symbol (lib_id "nescontroller:90DegreePort") (at 125.73 76.2 0) (unit 1)
-    (in_bom yes) (on_board yes) (fields_autoplaced)
-    (property "Reference" "U?" (id 0) (at 128.27 76.8349 0)
-      (effects (font (size 1.27 1.27)) (justify left))
-    )
-    (property "Value" "90DegreePort" (id 1) (at 128.27 79.3749 0)
-      (effects (font (size 1.27 1.27)) (justify left))
-    )
-    (property "Footprint" "port:NEScontrollerport" (id 2) (at 116.84 87.63 0)
+  (symbol (lib_id "nescontroller:90DegreePort") (at 38.1 105.41 0) (mirror y) (unit 1)
+    (in_bom yes) (on_board yes)
+    (property "Reference" "U2" (id 0) (at 46.99 111.76 0))
+    (property "Value" "90DegreePort" (id 1) (at 46.99 114.3 0))
+    (property "Footprint" "port:NEScontrollerport" (id 2) (at 46.99 116.84 0)
       (effects (font (size 1.27 1.27)) hide)
     )
-    (property "Datasheet" "" (id 3) (at 125.73 76.2 0)
+    (property "Datasheet" "" (id 3) (at 38.1 105.41 0)
       (effects (font (size 1.27 1.27)) hide)
     )
-    (pin "1")
-    (pin "2")
-    (pin "3")
-    (pin "4")
-    (pin "5")
+    (pin "5V")
+    (pin "C")
+    (pin "D")
+    (pin "G")
+    (pin "L")
   )
-  (symbol (lib_id "nescontroller:90DegreePort") (at 125.73 100.33 0) (unit 1)
-    (in_bom yes) (on_board yes) (fields_autoplaced)
-    (property "Reference" "U?" (id 0) (at 128.27 100.9649 0)
-      (effects (font (size 1.27 1.27)) (justify left))
-    )
-    (property "Value" "90DegreePort" (id 1) (at 128.27 103.5049 0)
-      (effects (font (size 1.27 1.27)) (justify left))
-    )
-    (property "Footprint" "port:NEScontrollerport" (id 2) (at 116.84 111.76 0)
+  (symbol (lib_name "90DegreePort_1") (lib_id "nescontroller:90DegreePort") (at 38.1 69.85 0) (mirror y) (unit 1)
+    (in_bom yes) (on_board yes)
+    (property "Reference" "U1" (id 0) (at 45.72 77.47 0))
+    (property "Value" "90DegreePort" (id 1) (at 45.72 80.01 0))
+    (property "Footprint" "port:NEScontrollerport" (id 2) (at 46.99 81.28 0)
       (effects (font (size 1.27 1.27)) hide)
     )
-    (property "Datasheet" "" (id 3) (at 125.73 100.33 0)
+    (property "Datasheet" "" (id 3) (at 38.1 69.85 0)
       (effects (font (size 1.27 1.27)) hide)
     )
-    (pin "1")
-    (pin "2")
-    (pin "3")
-    (pin "4")
-    (pin "5")
+    (pin "5V")
+    (pin "C")
+    (pin "D")
+    (pin "G")
+    (pin "L")
   )
   (sheet_instances
@@
   )
   (symbol_instances
+    (path "/9b419b92-e7b1-4b97-bdf9-f5d2605d9cad"
+      (reference "U1") (unit 1) (value "90DegreePort") (footprint "port:NEScontrollerport")
+    )
+    (path "/145fb29c-33d7-4c4d-bbec-1a96f9463fa1"
+      (reference "U2") (unit 1) (value "90DegreePort") (footprint "port:NEScontrollerport")
+    )
     (path "/00000000-0000-0000-0000-0000632cf335"
-      (reference "U?") (unit 1) (value "ProMicro") (footprint "")
-    )
-    (path "/9b419b92-e7b1-4b97-bdf9-f5d2605d9cad"
-      (reference "U?") (unit 1) (value "90DegreePort") (footprint "port:NEScontrollerport")
-    )
-    (path "/b4b95eb2-278e-4393-a446-0768c0bd5869"
-      (reference "U?") (unit 1) (value "90DegreePort") (footprint "port:NEScontrollerport")
+      (reference "U3") (unit 1) (value "ProMicro") (footprint "promicro:ProMicro")
     )
   )
